File: schematic/massam/R6502.kicad_sch (KiCad schematic)
At the start: 15 parts, among them U100A R6502, U101A SST39SF512, U102A UT62256PC-70LL, U103A GAL20L8, X100A 1.8Mhz

Commit message: added CPU_TEST dir
Connections:
- net GND: no longer U101A.3 (A15)
- net VCC: now also U101A.3 (A15)
Changed lines of the file:
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@@
   (junction (at 275.59 99.06) (diameter 0) (color 0 0 0 0)
+  )
+  (junction (at 124.46 100.33) (diameter 0) (color 0 0 0 0)
   )
   (junction (at 125.73 22.86) (diameter 0) (color 0 0 0 0)
@@
     (stroke (width 0) (type default) (color 0 0 0 0))
   )
+  (wire (pts (xy 124.46 100.33) (xy 115.57 100.33))
+    (stroke (width 0) (type default) (color 0 0 0 0))
+  )
   (wire (pts (xy 99.06 25.4) (xy 109.22 25.4))
     (stroke (width 0) (type default) (color 0 0 0 0))
@@
     (stroke (width 0) (type default) (color 0 0 0 0))
   )
-  (wire (pts (xy 124.46 87.63) (xy 124.46 92.71))
-    (stroke (width 0) (type default) (color 0 0 0 0))
-  )
-  (wire (pts (xy 132.08 100.33) (xy 132.08 97.79))
+  (wire (pts (xy 115.57 100.33) (xy 115.57 91.44))
     (stroke (width 0) (type default) (color 0 0 0 0))
   )
@@
     (stroke (width 0) (type default) (color 0 0 0 0))
   )
+  (wire (pts (xy 124.46 87.63) (xy 124.46 100.33))
+    (stroke (width 0) (type default) (color 0 0 0 0))
+  )
   (bus (pts (xy 119.38 55.88) (xy 119.38 58.42))
     (stroke (width 0) (type default) (color 0 0 0 0))
@@
     (stroke (width 0) (type default) (color 0 0 0 0))
   )
-  (wire (pts (xy 137.16 100.33) (xy 132.08 100.33))
+  (wire (pts (xy 137.16 100.33) (xy 124.46 100.33))
     (stroke (width 0) (type default) (color 0 0 0 0))
   )
@@
     )
     (property "Datasheet" "" (id 3) (at 99.06 19.05 0)
-      (effects (font (size 1.27 1.27)) hide)
-    )
-    (pin "1")
-  )
-  (symbol (lib_id "power:GNDREF") (at 124.46 92.71 0) (unit 1)
-    (in_bom yes) (on_board yes) (fields_autoplaced)
-    (property "Reference" "#PWR?" (id 0) (at 124.46 99.06 0)
-      (effects (font (size 1.27 1.27)) hide)
-    )
-    (property "Value" "GNDREF" (id 1) (at 124.46 97.2725 0))
-    (property "Footprint" "" (id 2) (at 124.46 92.71 0)
-      (effects (font (size 1.27 1.27)) hide)
-    )
-    (property "Datasheet" "" (id 3) (at 124.46 92.71 0)
       (effects (font (size 1.27 1.27)) hide)
     )
@@
     (pin "1")
   )
-  (symbol (lib_id "power:VCC") (at 132.08 97.79 0) (unit 1)
+  (symbol (lib_id "power:VCC") (at 115.57 91.44 0) (unit 1)
     (in_bom yes) (on_board yes)
-    (property "Reference" "#PWR?" (id 0) (at 132.08 101.6 0)
-      (effects (font (size 1.27 1.27)) hide)
-    )
-    (property "Value" "VCC" (id 1) (at 132.08 94.1855 0))
-    (property "Footprint" "" (id 2) (at 132.08 97.79 0)
-      (effects (font (size 1.27 1.27)) hide)
-    )
-    (property "Datasheet" "" (id 3) (at 132.08 97.79 0)
-      (effects (font (size 1.27 1.27)) hide)
-    )
+    (property "Reference" "#PWR?" (id 0) (at 115.57 95.25 0)
+      (effects (font (size 1.27 1.27)) hide)
+    )
+    (property "Value" "VCC" (id 1) (at 115.57 87.8355 0))
+    (property "Footprint" "" (id 2) (at 115.57 91.44 0)
+      (effects (font (size 1.27 1.27)) hide)
+    )
+    (property "Datasheet" "" (id 3) (at 115.57 91.44 0)
+      (effects (font (size 1.27 1.27)) hide)
+    )

Commit message: msbasic running OK...
Connections:
- net /RAMOE renamed /OE
- net /OE: now also U101A.24 (OE)
- net /ROMOE: no longer names the net of U103A.17 (IO17)
- net /ROMOE: no longer U101A.24 (OE)
Changed lines of the file:
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@@
-    (stroke (width 0) (type default) (color 0 0 0 0))
-  )
-  (wire (pts (xy 50.8 62.23) (xy 53.34 62.23))
     (stroke (width 0) (type default) (color 0 0 0 0))
   )
@@
     )
   )
-  (global_label "{slash}RAMOE" (shape input) (at 113.03 78.74 0) (fields_autoplaced)
-    (effects (font (size 1.27 1.27)) (justify left))
-    (property "Intersheet References" "${INTERSHEET_REFS}" (id 0) (at 123.0631 78.6606 0)
+  (global_label "{slash}OE" (shape input) (at 113.03 78.74 0) (fields_autoplaced)
+    (effects (font (size 1.27 1.27)) (justify left))
+    (property "Intersheet References" "${INTERSHEET_REFS}" (id 0) (at 119.2531 78.6606 0)
       (effects (font (size 1.27 1.27)) (justify left) hide)
     )
@@
     )
   )
-  (global_label "{slash}RAMOE" (shape input) (at 63.5 59.69 0) (fields_autoplaced)
-    (effects (font (size 1.27 1.27)) (justify left))
-    (property "Intersheet References" "${INTERSHEET_REFS}" (id 0) (at 73.5331 59.6106 0)
+  (global_label "{slash}OE" (shape input) (at 63.5 59.69 0) (fields_autoplaced)
+    (effects (font (size 1.27 1.27)) (justify left))
+    (property "Intersheet References" "${INTERSHEET_REFS}" (id 0) (at 69.7231 59.6106 0)
       (effects (font (size 1.27 1.27)) (justify left) hide)
     )
@@
     )
   )
-  (global_label "{slash}ROMOE" (shape input) (at 124.46 111.76 180) (fields_autoplaced)
+  (global_label "{slash}OE" (shape input) (at 124.46 111.76 180) (fields_autoplaced)
     (effects (font (size 1.27 1.27)) (justify right))
-    (property "Intersheet References" "${INTERSHEET_REFS}" (id 0) (at 114.185 111.6806 0)
+    (property "Intersheet References" "${INTERSHEET_REFS}" (id 0) (at 118.2369 111.6806 0)
       (effects (font (size 1.27 1.27)) (justify right) hide)
     )
   )
-  (global_label "{slash}RAMOE" (shape input) (at 261.62 109.22 90) (fields_autoplaced)
-    (effects (font (size 1.27 1.27)) (justify left))
-    (property "Intersheet References" "${INTERSHEET_REFS}" (id 0) (at 261.5406 99.1869 90)
+  (global_label "{slash}OE" (shape input) (at 261.62 109.22 90) (fields_autoplaced)
+    (effects (font (size 1.27 1.27)) (justify left))
+    (property "Intersheet References" "${INTERSHEET_REFS}" (id 0) (at 261.5406 102.9969 90)
       (effects (font (size 1.27 1.27)) (justify left) hide)
     )
@@
       (effects (font (size 1.27 1.27)) (justify left) hide)
     )
-  )
-  (global_label "{slash}ROMOE" (shape input) (at 53.34 62.23 0) (fields_autoplaced)
-    (effects (font (size 1.27 1.27)) (justify left))
-    (property "Intersheet References" "${INTERSHEET_REFS}" (id 0) (at 63.615 62.3094 0)
-      (effects (font (size 1.27 1.27)) (justify left) hide)
-    )

Commit message: Fix R6502 R/W signal to slot
Connections:
- net R/W: no longer J?.b24 (Pin_b24)
- net /RAMWE renamed /WE
- net /WE: now also J?.b24 (Pin_b24)
Changed lines of the file:
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@@
   (junction (at 224.79 111.76) (diameter 0) (color 0 0 0 0)
-  )
-  (junction (at 215.9 97.79) (diameter 0) (color 0 0 0 0)
   )
   (junction (at 20.32 80.01) (diameter 0) (color 0 0 0 0)
@@
     (stroke (width 0) (type default) (color 0 0 0 0))
   )
-  (wire (pts (xy 214.63 97.79) (xy 215.9 97.79))
+  (wire (pts (xy 214.63 97.79) (xy 217.17 97.79))
     (stroke (width 0) (type default) (color 0 0 0 0))
   )
@@
     (stroke (width 0) (type default) (color 0 0 0 0))
   )
+  (wire (pts (xy 252.73 160.02) (xy 257.81 160.02))
+    (stroke (width 0) (type default) (color 0 0 0 0))
+  )
   (wire (pts (xy 264.16 97.79) (xy 264.16 153.67))
     (stroke (width 0) (type default) (color 0 0 0 0))
@@
     (stroke (width 0) (type default) (color 0 0 0 0))
   )
-  (wire (pts (xy 215.9 97.79) (xy 215.9 152.4))
-    (stroke (width 0) (type default) (color 0 0 0 0))
-  )
   (wire (pts (xy 275.59 83.82) (xy 275.59 86.36))
     (stroke (width 0) (type default) (color 0 0 0 0))
@@
     (stroke (width 0) (type default) (color 0 0 0 0))
   )
-  (wire (pts (xy 257.81 107.95) (xy 257.81 152.4))
-    (stroke (width 0) (type default) (color 0 0 0 0))
-  )
   (wire (pts (xy 252.73 120.65) (xy 269.24 120.65))
     (stroke (width 0) (type default) (color 0 0 0 0))
@@
     (stroke (width 0) (type default) (color 0 0 0 0))
   )
-  (wire (pts (xy 215.9 97.79) (xy 217.17 97.79))
-    (stroke (width 0) (type default) (color 0 0 0 0))
-  )
   (wire (pts (xy 172.72 110.49) (xy 165.1 110.49))
     (stroke (width 0) (type default) (color 0 0 0 0))
@@
     (stroke (width 0) (type default) (color 0 0 0 0))
   )
-  (wire (pts (xy 257.81 152.4) (xy 215.9 152.4))
-    (stroke (width 0) (type default) (color 0 0 0 0))
-  )
   (bus (pts (xy 74.93 58.42) (xy 74.93 60.96))
     (stroke (width 0) (type default) (color 0 0 0 0))
@@
   )
   (wire (pts (xy 252.73 64.77) (xy 262.89 64.77))
+    (stroke (width 0) (type default) (color 0 0 0 0))
+  )
+  (wire (pts (xy 257.81 107.95) (xy 257.81 160.02))
     (stroke (width 0) (type default) (color 0 0 0 0))
   )
@@
     )
   )
-  (global_label "{slash}RAMWE" (shape input) (at 53.34 52.07 0) (fields_autoplaced)
+  (global_label "{slash}WE" (shape input) (at 53.34 52.07 0) (fields_autoplaced)
     (effects (font (size 1.27 1.27)) (justify left))
-    (property "Intersheet References" "${INTERSHEET_REFS}" (id 0) (at 63.4941 51.9906 0)
+    (property "Intersheet References" "${INTERSHEET_REFS}" (id 0) (at 59.6841 51.9906 0)
       (effects (font (size 1.27 1.27)) (justify left) hide)
     )
@@
     )
   )
-  (global_label "{slash}RAMWE" (shape input) (at 113.03 81.28 0) (fields_autoplaced)
+  (global_label "{slash}WE" (shape input) (at 113.03 81.28 0) (fields_autoplaced)
     (effects (font (size 1.27 1.27)) (justify left))
-    (property "Intersheet References" "${INTERSHEET_REFS}" (id 0) (at 123.1841 81.2006 0)
+    (property "Intersheet References" "${INTERSHEET_REFS}" (id 0) (at 119.3741 81.2006 0)
       (effects (font (size 1.27 1.27)) (justify left) hide)
     )
@@
     )
   )
+  (global_label "{slash}WE" (shape input) (at 252.73 160.02 180) (fields_autoplaced)
+    (effects (font (size 1.27 1.27)) (justify right))
+    (property "Intersheet References" "${INTERSHEET_REFS}" (id 0) (at 246.3859 160.0994 0)
+      (effects (font (size 1.27 1.27)) (justify right) hide)
+    )
+  )
