File: schematic/massam/W65C02.kicad_sch (KiCad schematic)
At the start: 26 parts, among them U100B W65C02SxPL, U101B SST39SF512, U102B UT62256PC-70LL, U103B GAL20L8, U104B 74AHC04, Y100B 14.310Mhz

Commit message: added CPU_TEST dir
Parts:
- removed R3: 33K, symbol Device:R
- R1, R2: value 1k8 -> 1k
Connections:
- net A15 is gone; now on net +5V: J?.b1 (Pin_b1), U100B.28 (A15), U101B.3 (A15), U103B.1 (I1)
- net +5V: now also U100B.42 (~{SO})
- net PHI2: now also U100B.41 (ϕ0)
- no-connect marks 9 -> 8
Changed lines of the file:
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@@
   (junction (at 45.72 80.01) (diameter 0) (color 0 0 0 0)
   )
-  (junction (at 19.05 132.08) (diameter 0) (color 0 0 0 0)
-  )
   (junction (at 55.88 175.26) (diameter 0) (color 0 0 0 0)
   )
@@
   (junction (at 30.48 175.26) (diameter 0) (color 0 0 0 0)
   )
+  (junction (at 107.95 88.9) (diameter 0) (color 0 0 0 0)
+  )
   (junction (at 137.16 167.64) (diameter 0) (color 0 0 0 0)
   )
@@
   )
   (no_connect (at 114.3 78.74))
+  (no_connect (at 187.96 55.88))
   (no_connect (at 114.3 81.28))
   (no_connect (at 114.3 83.82))
   (no_connect (at 187.96 83.82))
-  (no_connect (at 187.96 50.8))
   (no_connect (at 187.96 53.34))
   (no_connect (at 187.96 81.28))
   (no_connect (at 187.96 86.36))
-  (no_connect (at 187.96 91.44))
   (bus_entry (at 265.43 110.49) (size -2.54 2.54)
     (stroke (width 0) (type default) (color 0 0 0 0))
@@
     (stroke (width 0) (type default) (color 0 0 0 0))
   )
-  (bus_entry (at 91.44 73.66) (size 2.54 2.54)
-    (stroke (width 0) (type default) (color 0 0 0 0))
-  )
   (bus_entry (at 220.98 40.64) (size -2.54 2.54)
     (stroke (width 0) (type default) (color 0 0 0 0))
@@
     (stroke (width 0) (type default) (color 0 0 0 0))
   )
-  (bus (pts (xy 186.69 55.88) (xy 187.96 55.88))
-    (stroke (width 0) (type default) (color 0 0 0 0))
-  )
   (wire (pts (xy 20.32 62.23) (xy 33.02 62.23))
     (stroke (width 0) (type default) (color 0 0 0 0))
@@
     (stroke (width 0) (type default) (color 0 0 0 0))
   )
-  (wire (pts (xy 114.3 88.9) (xy 101.6 88.9))
+  (wire (pts (xy 114.3 88.9) (xy 107.95 88.9))
     (stroke (width 0) (type default) (color 0 0 0 0))
   )
@@
     (stroke (width 0) (type default) (color 0 0 0 0))
   )
+  (wire (pts (xy 107.95 76.2) (xy 107.95 88.9))
+    (stroke (width 0) (type default) (color 0 0 0 0))
+  )
   (bus (pts (xy 91.44 118.11) (xy 91.44 120.65))
     (stroke (width 0) (type default) (color 0 0 0 0))
@@
     (stroke (width 0) (type default) (color 0 0 0 0))
   )
-  (wire (pts (xy 19.05 134.62) (xy 19.05 132.08))
-    (stroke (width 0) (type default) (color 0 0 0 0))
-  )
   (wire (pts (xy 171.45 193.04) (xy 171.45 194.31))
     (stroke (width 0) (type default) (color 0 0 0 0))
@@
     (stroke (width 0) (type default) (color 0 0 0 0))
   )
+  (wire (pts (xy 107.95 88.9) (xy 101.6 88.9))
+    (stroke (width 0) (type default) (color 0 0 0 0))
+  )
   (bus (pts (xy 220.98 26.67) (xy 91.44 26.67))
     (stroke (width 0) (type default) (color 0 0 0 0))
@@
     (stroke (width 0) (type default) (color 0 0 0 0))
   )
+  (wire (pts (xy 185.42 50.8) (xy 187.96 50.8))
+    (stroke (width 0) (type default) (color 0 0 0 0))
+  )
   (wire (pts (xy 276.86 158.75) (xy 276.86 160.02))
     (stroke (width 0) (type default) (color 0 0 0 0))
@@
     (stroke (width 0) (type default) (color 0 0 0 0))
   )
-  (wire (pts (xy 19.05 142.24) (xy 19.05 146.05))
-    (stroke (width 0) (type default) (color 0 0 0 0))
-  )
   (bus (pts (xy 91.44 35.56) (xy 91.44 38.1))
     (stroke (width 0) (type default) (color 0 0 0 0))
@@
     (stroke (width 0) (type default) (color 0 0 0 0))
   )
+  (wire (pts (xy 107.95 76.2) (xy 114.3 76.2))
+    (stroke (width 0) (type default) (color 0 0 0 0))
+  )
   (wire (pts (xy 248.92 49.53) (xy 259.08 49.53))
     (stroke (width 0) (type default) (color 0 0 0 0))
@@
     (stroke (width 0) (type default) (color 0 0 0 0))
   )
+  (wire (pts (xy 172.72 91.44) (xy 172.72 83.82))
+    (stroke (width 0) (type default) (color 0 0 0 0))
+  )
   (wire (pts (xy 248.92 115.57) (xy 262.89 115.57))
     (stroke (width 0) (type default) (color 0 0 0 0))
@@
     (stroke (width 0) (type default) (color 0 0 0 0))
   )
-  (wire (pts (xy 93.98 76.2) (xy 114.3 76.2))
-    (stroke (width 0) (type default) (color 0 0 0 0))
-  )
   (wire (pts (xy 29.21 69.85) (xy 33.02 69.85))
     (stroke (width 0) (type default) (color 0 0 0 0))
@@
     (stroke (width 0) (type default) (color 0 0 0 0))
   )
-  (bus (pts (xy 91.44 73.66) (xy 91.44 118.11))
+  (bus (pts (xy 91.44 71.12) (xy 91.44 118.11))
     (stroke (width 0) (type default) (color 0 0 0 0))
   )
@@
     (stroke (width 0) (type default) (color 0 0 0 0))
   )
-  (bus (pts (xy 91.44 71.12) (xy 91.44 73.66))
-    (stroke (width 0) (type default) (color 0 0 0 0))
-  )
   (bus (pts (xy 153.67 35.56) (xy 153.67 38.1))
     (stroke (width 0) (type default) (color 0 0 0 0))
@@
   )
   (wire (pts (xy 129.54 179.07) (xy 129.54 181.61))
+    (stroke (width 0) (type default) (color 0 0 0 0))
+  )
+  (wire (pts (xy 187.96 91.44) (xy 172.72 91.44))
     (stroke (width 0) (type default) (color 0 0 0 0))
   )
@@
     )
   )
-  (global_label "PHI2" (shape input) (at 186.69 55.88 180) (fields_autoplaced)
+  (global_label "PHI2" (shape input) (at 185.42 50.8 180) (fields_autoplaced)
     (effects (font (size 1.27 1.27)) (justify right))
-    (property "Intersheet References" "${INTERSHEET_REFS}" (id 0) (at 179.8621 55.8006 0)
+    (property "Intersheet References" "${INTERSHEET_REFS}" (id 0) (at 178.5921 50.7206 0)
       (effects (font (size 1.27 1.27)) (justify right) hide)
     )
@@
       (effects (font (size 1.27 1.27)) (justify right) hide)
     )
-  )
-  (symbol (lib_id "power:GNDREF") (at 19.05 146.05 0) (unit 1)
-    (in_bom yes) (on_board yes)
-    (property "Reference" "#PWR?" (id 0) (at 19.05 152.4 0)
-      (effects (font (size 1.27 1.27)) hide)
-    )
-    (property "Value" "GNDREF" (id 1) (at 21.59 146.05 90))
-    (property "Footprint" "" (id 2) (at 19.05 146.05 0)
-      (effects (font (size 1.27 1.27)) hide)
-    )
-    (property "Datasheet" "" (id 3) (at 19.05 146.05 0)
-      (effects (font (size 1.27 1.27)) hide)
-    )
-    (pin "1")
   )
   (symbol (lib_id "Device:C") (at 44.45 182.88 0) (unit 1)
@@
     (in_bom yes) (on_board yes)
     (property "Reference" "R2" (id 0) (at 48.26 111.76 90))
-    (property "Value" "1k8" (id 1) (at 55.88 111.76 90))
+    (property "Value" "1k" (id 1) (at 55.88 111.76 90))
     (property "Footprint" "" (id 2) (at 52.07 114.808 90)
       (effects (font (size 1.27 1.27)) hide)
     )
     (property "Datasheet" "~" (id 3) (at 52.07 113.03 0)
-      (effects (font (size 1.27 1.27)) hide)
-    )
-    (pin "1")
-    (pin "2")
-  )
-  (symbol (lib_id "Device:R") (at 19.05 138.43 0) (unit 1)
-    (in_bom yes) (on_board yes)
-    (property "Reference" "R3" (id 0) (at 20.32 134.62 90))
-    (property "Value" "33K" (id 1) (at 20.32 142.24 90))
-    (property "Footprint" "" (id 2) (at 17.272 138.43 90)
-      (effects (font (size 1.27 1.27)) hide)
-    )
-    (property "Datasheet" "~" (id 3) (at 19.05 138.43 0)
       (effects (font (size 1.27 1.27)) hide)
     )
@@
     (pin "7")
   )
+  (symbol (lib_id "power:+5V") (at 172.72 83.82 0) (unit 1)
+    (in_bom yes) (on_board yes) (fields_autoplaced)
+    (property "Reference" "#PWR?" (id 0) (at 172.72 87.63 0)
+      (effects (font (size 1.27 1.27)) hide)
+    )
+    (property "Value" "+5V" (id 1) (at 172.72 78.74 0))
+    (property "Footprint" "" (id 2) (at 172.72 83.82 0)
+      (effects (font (size 1.27 1.27)) hide)
+    )
+    (property "Datasheet" "" (id 3) (at 172.72 83.82 0)
+      (effects (font (size 1.27 1.27)) hide)
+    )
+    (pin "1")
+  )
   (symbol (lib_id "power:+5V") (at 130.81 114.3 0) (unit 1)
     (in_bom yes) (on_board yes) (fields_autoplaced)
@@
     (in_bom yes) (on_board yes)
     (property "Reference" "R1" (id 0) (at 26.67 111.76 90))
-    (property "Value" "1k8" (id 1) (at 34.29 111.76 90))
+    (property "Value" "1k" (id 1) (at 34.29 111.76 90))
     (property "Footprint" "" (id 2) (at 30.48 114.808 90)
       (effects (font (size 1.27 1.27)) hide)

Commit message: msbasic running OK...
Connections:
- net /SLOT0 is gone; now on net /OE: U103B.18 (IO18)
- net /SLOT3 is gone; now on net /SLOT2: U103B.15 (IO15)
- net RESET: now also U103B.16 (IO16)
- net R/W: no longer J?.b24 (Pin_b24), U102B.27 (~{WE})
- net /RAMCS: now also U103B.19 (IO19); no longer U103B.21 (IO21)
- net /SLOT2: no longer U103B.16 (IO16)
- net /RD renamed /OE
- net /OE: no longer U103B.19 (IO19)
- net /SLOT1: no longer names the net of U103B.17 (IO17)
- new net /WE: J?.b24 (Pin_b24), U102B.27 (~{WE}), U103B.21 (IO21)
Changed lines of the file:
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@@
   (junction (at 45.72 80.01) (diameter 0) (color 0 0 0 0)
   )
+  (junction (at 165.1 151.13) (diameter 0) (color 0 0 0 0)
+  )
   (junction (at 55.88 175.26) (diameter 0) (color 0 0 0 0)
   )
@@
   (junction (at 67.31 190.5) (diameter 0) (color 0 0 0 0)
   )
-  (junction (at 148.59 107.95) (diameter 0) (color 0 0 0 0)
-  )
   (junction (at 77.47 190.5) (diameter 0) (color 0 0 0 0)
   )
@@
   )
   (junction (at 156.21 148.59) (diameter 0) (color 0 0 0 0)
-  )
-  (junction (at 161.29 151.13) (diameter 0) (color 0 0 0 0)
   )
   (junction (at 91.44 26.67) (diameter 0) (color 0 0 0 0)
@@
     (stroke (width 0) (type default) (color 0 0 0 0))
   )
+  (wire (pts (xy 165.1 134.62) (xy 165.1 151.13))
+    (stroke (width 0) (type default) (color 0 0 0 0))
+  )
   (bus (pts (xy 261.62 59.69) (xy 261.62 62.23))
     (stroke (width 0) (type default) (color 0 0 0 0))
@@
     (stroke (width 0) (type default) (color 0 0 0 0))
   )
-  (wire (pts (xy 161.29 151.13) (xy 254 151.13))
+  (wire (pts (xy 143.51 151.13) (xy 165.1 151.13))
     (stroke (width 0) (type default) (color 0 0 0 0))
   )
@@
     (stroke (width 0) (type default) (color 0 0 0 0))
   )
+  (wire (pts (xy 165.1 151.13) (xy 254 151.13))
+    (stroke (width 0) (type default) (color 0 0 0 0))
+  )
   (wire (pts (xy 139.7 193.04) (xy 139.7 194.31))
     (stroke (width 0) (type default) (color 0 0 0 0))
@@
     (stroke (width 0) (type default) (color 0 0 0 0))
   )
-  (wire (pts (xy 143.51 151.13) (xy 161.29 151.13))
-    (stroke (width 0) (type default) (color 0 0 0 0))
-  )
   (wire (pts (xy 248.92 72.39) (xy 259.08 72.39))
     (stroke (width 0) (type default) (color 0 0 0 0))
@@
     (stroke (width 0) (type default) (color 0 0 0 0))
   )
-  (wire (pts (xy 148.59 107.95) (xy 161.29 107.95))
-    (stroke (width 0) (type default) (color 0 0 0 0))
-  )
   (wire (pts (xy 208.28 63.5) (xy 218.44 63.5))
     (stroke (width 0) (type default) (color 0 0 0 0))
@@
     (stroke (width 0) (type default) (color 0 0 0 0))
   )
-  (wire (pts (xy 161.29 107.95) (xy 161.29 151.13))
-    (stroke (width 0) (type default) (color 0 0 0 0))
-  )
   (bus (pts (xy 20.32 46.99) (xy 20.32 49.53))
     (stroke (width 0) (type default) (color 0 0 0 0))
@@
   )
   (wire (pts (xy 257.81 97.79) (xy 257.81 148.59))
-    (stroke (width 0) (type default) (color 0 0 0 0))
-  )
-  (wire (pts (xy 58.42 52.07) (xy 66.04 52.07))
     (stroke (width 0) (type default) (color 0 0 0 0))
   )
@@
     (effects (font (size 1.27 1.27)) (justify right bottom))
   )
-  (label "{slash}WR" (at 248.92 95.25 0)
+  (label "{slash}WE" (at 248.92 95.25 0)
     (effects (font (size 1.27 1.27)) (justify left bottom))
   )
@@
     (effects (font (size 1.27 1.27)) (justify left bottom))
   )
-  (label "{slash}RD" (at 248.92 97.79 0)
+  (label "{slash}RD_OE" (at 248.92 97.79 0)
     (effects (font (size 1.27 1.27)) (justify left bottom))
   )
@@
     )
   )
-  (global_label "{slash}RAMCS" (shape input) (at 66.04 41.91 0) (fields_autoplaced)
+  (global_label "{slash}WE" (shape input) (at 66.04 41.91 0) (fields_autoplaced)
     (effects (font (size 1.27 1.27)) (justify left))
-    (property "Intersheet References" "${INTERSHEET_REFS}" (id 0) (at 76.0731 41.8306 0)
+    (property "Intersheet References" "${INTERSHEET_REFS}" (id 0) (at 72.3841 41.8306 0)
       (effects (font (size 1.27 1.27)) (justify left) hide)
     )
@@
     )
   )
-  (global_label "{slash}SLOT1" (shape input) (at 66.04 52.07 0) (fields_autoplaced)
-    (effects (font (size 1.27 1.27)) (justify left))
-    (property "Intersheet References" "${INTERSHEET_REFS}" (id 0) (at 75.5288 51.9906 0)
-      (effects (font (size 1.27 1.27)) (justify left) hide)
-    )
-  )
   (global_label "PHI2" (shape input) (at 20.32 62.23 180) (fields_autoplaced)
     (effects (font (size 1.27 1.27)) (justify right))
@@
     )
   )
-  (global_label "{slash}SLOT2" (shape input) (at 80.01 54.61 0) (fields_autoplaced)
+  (global_label "RESET" (shape input) (at 80.01 54.61 0) (fields_autoplaced)
     (effects (font (size 1.27 1.27)) (justify left))
-    (property "Intersheet References" "${INTERSHEET_REFS}" (id 0) (at 89.4988 54.5306 0)
+    (property "Intersheet References" "${INTERSHEET_REFS}" (id 0) (at 88.1683 54.5306 0)
       (effects (font (size 1.27 1.27)) (justify left) hide)
     )
@@
     )
   )
-  (global_label "{slash}SLOT0" (shape input) (at 80.01 49.53 0) (fields_autoplaced)
+  (global_label "{slash}OE" (shape input) (at 80.01 49.53 0) (fields_autoplaced)
     (effects (font (size 1.27 1.27)) (justify left))
-    (property "Intersheet References" "${INTERSHEET_REFS}" (id 0) (at 89.4988 49.4506 0)
+    (property "Intersheet References" "${INTERSHEET_REFS}" (id 0) (at 86.2331 49.4506 0)
       (effects (font (size 1.27 1.27)) (justify left) hide)
     )
   )
-  (global_label "{slash}RD" (shape input) (at 161.29 104.14 0) (fields_autoplaced)
+  (global_label "{slash}OE" (shape input) (at 161.29 104.14 0) (fields_autoplaced)
     (effects (font (size 1.27 1.27)) (justify left))
-    (property "Intersheet References" "${INTERSHEET_REFS}" (id 0) (at 167.5736 104.0606 0)
+    (property "Intersheet References" "${INTERSHEET_REFS}" (id 0) (at 167.5131 104.0606 0)
       (effects (font (size 1.27 1.27)) (justify left) hide)
     )
@@
     )
   )
-  (global_label "{slash}RD" (shape input) (at 66.04 46.99 0) (fields_autoplaced)
+  (global_label "{slash}RAMCS" (shape input) (at 66.04 46.99 0) (fields_autoplaced)
     (effects (font (size 1.27 1.27)) (justify left))
-    (property "Intersheet References" "${INTERSHEET_REFS}" (id 0) (at 72.3236 46.9106 0)
+    (property "Intersheet References" "${INTERSHEET_REFS}" (id 0) (at 76.0731 46.9106 0)
       (effects (font (size 1.27 1.27)) (justify left) hide)
     )
@@
     )
   )
-  (global_label "{slash}SLOT3" (shape input) (at 66.04 57.15 0) (fields_autoplaced)
+  (global_label "{slash}SLOT2" (shape input) (at 66.04 57.15 0) (fields_autoplaced)
     (effects (font (size 1.27 1.27)) (justify left))
     (property "Intersheet References" "${INTERSHEET_REFS}" (id 0) (at 75.5288 57.0706 0)
       (effects (font (size 1.27 1.27)) (justify left) hide)
     )
+  )
+  (global_label "{slash}WE" (shape input) (at 165.1 134.62 90) (fields_autoplaced)
+    (effects (font (size 1.27 1.27)) (justify left))
+    (property "Intersheet References" "${INTERSHEET_REFS}" (id 0) (at 165.0206 128.2759 90)
+      (effects (font (size 1.27 1.27)) (justify left) hide)
+    )

Commit message: Alinhamento com biosmon
Parts:
- added C105B?: 18pF, symbol Device:C
- added C105B?: 36pF, symbol Device:C
- added L1: 220uH, symbol Device:L
- added Q?: 2N2222A, Package_TO_SOT_THT:TO-39-3, symbol Transistor_BJT:2N2219
- added R?: 100R, symbol Device:R
- added R?: 47K, symbol Device:R
- added Y100B?: 14.310Mhz, symbol Device:Crystal
Connections:
- net +5V: now also L1.1
- net A7: now also U103B.23 (I23)
- net GND: now also C105B?.2, C105B?.2, Q?.1 (E); no longer U103B.11 (I11), U103B.23 (I23)
- net PHI2: now also R?.2; no longer R2.2, U104B.4, Y100B.2
- net RESET: no longer U103B.16 (IO16)
- net /IORQ: now also U103B.11 (I11)
- net at U104B.5: now also R2.2, U104B.4, Y100B.2
- new net: C105B?.1, L1.2, Q?.3 (C), R?.1, R?.2, Y100B?.2
- new net: C105B?.1, Q?.2 (B), R?.1, Y100B?.1
Other:
- moved on the sheet: R1, R2, U104BA, U104BB, U104BC, Y100B
