File: schematic/massam/serialInterface.kicad_sch (KiCad schematic)
At the start: 18 parts, among them J200 Conn_02x40_Row_Letter_First, J201 RS232, U200 16550, U201 74LS138, U202 MAX232

Commit message: Added schematic for W65C02
Other:
- title: SPARTAN -> HMC56
Changed lines of the file:
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@@
   (paper "A4")
   (title_block
-    (title "SPARTAN")
+    (title "HMC56")
     (date "2024-02-11")
     (rev "A")
     (company "Open Software")
-    (comment 1 "Retro computer SPARTAN using 65C02")
+    (comment 1 "Retro computer HMC56 using R6502")
     (comment 2 "Paulo da Silva (pdsilva)")
     (comment 3 "ppsilv gmail com")

Commit message: added CPU_TEST dir
Connections:
- net at U202.13 (R1IN): now also J201.2; no longer J201.3
- net at U202.14 (T1OUT): now also J201.3; no longer J201.2
Other:
- note added: "DTE(Data terminal equipment) Master as PC"
Changed lines of the file:
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@@
-    (stroke (width 0) (type default) (color 0 0 0 0))
-  )
-  (wire (pts (xy 238.76 82.55) (xy 257.81 82.55))
     (stroke (width 0) (type default) (color 0 0 0 0))
   )
@@
     (stroke (width 0) (type default) (color 0 0 0 0))
   )
-  (wire (pts (xy 257.81 80.01) (xy 266.7 80.01))
-    (stroke (width 0) (type default) (color 0 0 0 0))
-  )
   (wire (pts (xy 43.18 163.83) (xy 118.11 163.83))
     (stroke (width 0) (type default) (color 0 0 0 0))
@@
     (stroke (width 0) (type default) (color 0 0 0 0))
   )
-  (wire (pts (xy 257.81 74.93) (xy 266.7 74.93))
-    (stroke (width 0) (type default) (color 0 0 0 0))
-  )
   (wire (pts (xy 143.51 30.48) (xy 182.88 30.48))
     (stroke (width 0) (type default) (color 0 0 0 0))
@@
     (stroke (width 0) (type default) (color 0 0 0 0))
   )
+  (wire (pts (xy 243.84 72.39) (xy 238.76 72.39))
+    (stroke (width 0) (type default) (color 0 0 0 0))
+  )
   (wire (pts (xy 113.03 133.35) (xy 113.03 130.81))
     (stroke (width 0) (type default) (color 0 0 0 0))
@@
     (stroke (width 0) (type default) (color 0 0 0 0))
   )
-  (wire (pts (xy 238.76 72.39) (xy 257.81 72.39))
-    (stroke (width 0) (type default) (color 0 0 0 0))
-  )
   (wire (pts (xy 238.76 46.99) (xy 245.11 46.99))
     (stroke (width 0) (type default) (color 0 0 0 0))
@@
     (stroke (width 0) (type default) (color 0 0 0 0))
   )
+  (wire (pts (xy 243.84 80.01) (xy 243.84 72.39))
+    (stroke (width 0) (type default) (color 0 0 0 0))
+  )
   (wire (pts (xy 39.37 156.21) (xy 118.11 156.21))
     (stroke (width 0) (type default) (color 0 0 0 0))
@@
     (stroke (width 0) (type default) (color 0 0 0 0))
   )
+  (wire (pts (xy 243.84 80.01) (xy 266.7 80.01))
+    (stroke (width 0) (type default) (color 0 0 0 0))
+  )
   (wire (pts (xy 20.32 90.17) (xy 21.59 90.17))
     (stroke (width 0) (type default) (color 0 0 0 0))
@@
     (stroke (width 0) (type default) (color 0 0 0 0))
   )
+  (wire (pts (xy 262.89 74.93) (xy 266.7 74.93))
+    (stroke (width 0) (type default) (color 0 0 0 0))
+  )
   (wire (pts (xy 34.29 49.53) (xy 44.45 49.53))
     (stroke (width 0) (type default) (color 0 0 0 0))
@@
     (stroke (width 0) (type default) (color 0 0 0 0))
   )
+  (wire (pts (xy 238.76 82.55) (xy 262.89 82.55))
+    (stroke (width 0) (type default) (color 0 0 0 0))
+  )
   (bus (pts (xy 46.99 46.99) (xy 46.99 49.53))
     (stroke (width 0) (type default) (color 0 0 0 0))
@@
     (stroke (width 0) (type default) (color 0 0 0 0))
   )
-  (wire (pts (xy 257.81 82.55) (xy 257.81 80.01))
-    (stroke (width 0) (type default) (color 0 0 0 0))
-  )
   (wire (pts (xy 220.98 130.81) (xy 233.68 130.81))
     (stroke (width 0) (type default) (color 0 0 0 0))
@@
     (stroke (width 0) (type default) (color 0 0 0 0))
   )
+  (wire (pts (xy 262.89 82.55) (xy 262.89 74.93))
+    (stroke (width 0) (type default) (color 0 0 0 0))
+  )
   (bus (pts (xy 46.99 50.8) (xy 46.99 64.77))
     (stroke (width 0) (type default) (color 0 0 0 0))
@@
     (stroke (width 0) (type default) (color 0 0 0 0))
   )
-  (wire (pts (xy 257.81 72.39) (xy 257.81 74.93))
-    (stroke (width 0) (type default) (color 0 0 0 0))
-  )
   (wire (pts (xy 243.84 62.23) (xy 243.84 67.31))
     (stroke (width 0) (type default) (color 0 0 0 0))
   )
+  (text "DTE(Data terminal equipment)\nMaster as PC" (at 250.19 57.15 0)
+    (effects (font (size 1.5 1.5)) (justify left bottom))
+  )
   (label "A2" (at 34.29 67.31 0)

Commit message: Fixed max232 cap pin 2 was inverted
Connections:
- net GNDREF: no longer C205.2
- net VCC: now also C205.2
Other:
- moved on the sheet: C205

Commit message: Alinhamento com biosmon
Connections:
- net A15: no longer U201.6 (E3)
- net A8: no longer U201.1 (A0)
- net IO_02: no longer U201.13 (O2)
- net A5: now reaches J200.b5 (Pin_b5)
- net A5: now also U201.2 (A1)
- net A10 renamed A6
- net A9 renamed A7
- net A7: no longer U201.2 (A1)
- new net A08: U201.6 (E3)
- new net A4: U201.1 (A0)
- new net VDPCS: U201.13 (O2)
Other:
- note added: "IORQ Address: FF0x <-> FF7x"
